File: Rudi-NX Mark II/Rudi_updatedschem_Nov_14/Rudi_updatedschem_Nov_14.kicad_pcb (KiCad board)
At the start: 4 copper layers, 82.6 x 66 mm, 18 parts, among them J10 TFM-120-02-L-D-WT-K-TR

Commit message: done
Routing:
- net GND: track 6.55 -> 84.6 mm
- net +5V: track 48.9 -> 75.8 mm
Changed lines of the file:
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@@
     (fp_circle (center 0 0) (end 3.2 0) (layer "Cmts.User") (width 0.15) (fill none))
     (fp_circle (center 0 0) (end 3.45 0) (layer "F.CrtYd") (width 0.05) (fill none))
+    (pad "1" connect circle (at 0 0) (size 6.4 6.4) (layers "F.Cu" "F.Mask"))
+    (pad "1" thru_hole circle (at 0 0) (size 3.6 3.6) (drill 3.2) (layers *.Cu *.Mask))
     (pad "1" connect circle (at 0 0) (size 6.4 6.4) (layers "B.Cu" "B.Mask"))
-    (pad "1" thru_hole circle (at 0 0) (size 3.6 3.6) (drill 3.2) (layers *.Cu *.Mask))
-    (pad "1" connect circle (at 0 0) (size 6.4 6.4) (layers "F.Cu" "F.Mask"))
   )
   (footprint "Connector_JST:JST_XH_B4B-XH-A_1x04_P2.50mm_Vertical" (layer "F.Cu")
@@
     (fp_circle (center 0 0) (end 3.2 0) (layer "Cmts.User") (width 0.15) (fill none))
     (fp_circle (center 0 0) (end 3.45 0) (layer "F.CrtYd") (width 0.05) (fill none))
+    (pad "1" thru_hole circle (at 0 0) (size 3.6 3.6) (drill 3.2) (layers *.Cu *.Mask))
     (pad "1" connect circle (at 0 0) (size 6.4 6.4) (layers "B.Cu" "B.Mask"))
-    (pad "1" thru_hole circle (at 0 0) (size 3.6 3.6) (drill 3.2) (layers *.Cu *.Mask))
     (pad "1" connect circle (at 0 0) (size 6.4 6.4) (layers "F.Cu" "F.Mask"))
   )
@@
   (via (at 140.3 91.6) (size 0.8) (drill 0.4) (layers "F.Cu" "B.Cu") (net 5))
   (segment (start 144.145 94.805) (end 144.145 91.555) (width 0.25) (layer "F.Cu") (net 6))
+  (segment (start 112.285 105.43) (end 114.27 105.43) (width 0.25) (layer "F.Cu") (net 6))
+  (segment (start 117.2 81.3) (end 114.74 78.84) (width 0.25) (layer "F.Cu") (net 6))
+  (segment (start 113.14 88.84) (end 112.285 88.84) (width 0.25) (layer "F.Cu") (net 6))
+  (segment (start 114.27 105.43) (end 115.9 103.8) (width 0.25) (layer "F.Cu") (net 6))
+  (segment (start 112.285 110.43) (end 117.2 105.515) (width 0.25) (layer "F.Cu") (net 6))
+  (segment (start 115.9 103.8) (end 115.9 85.2) (width 0.25) (layer "F.Cu") (net 6))
+  (segment (start 115.9 85.2) (end 114.54 83.84) (width 0.25) (layer "F.Cu") (net 6))
   (segment (start 144.145 91.555) (end 144.2 91.5) (width 0.25) (layer "F.Cu") (net 6))
+  (segment (start 114.54 83.84) (end 112.285 83.84) (width 0.25) (layer "F.Cu") (net 6))
+  (segment (start 114.74 78.84) (end 112.285 78.84) (width 0.25) (layer "F.Cu") (net 6))
+  (segment (start 117.2 105.515) (end 117.2 81.3) (width 0.25) (layer "F.Cu") (net 6))
   (segment (start 161.925 98.235) (end 161.925 100.925) (width 0.25) (layer "F.Cu") (net 6))
+  (segment (start 112.285 100.43) (end 114.5 98.215) (width 0.25) (layer "F.Cu") (net 6))
   (segment (start 161.925 100.925) (end 162.3 101.3) (width 0.25) (layer "F.Cu") (net 6))
+  (segment (start 114.5 90.2) (end 113.14 88.84) (width 0.25) (layer "F.Cu") (net 6))
+  (segment (start 114.5 98.215) (end 114.5 90.2) (width 0.25) (layer "F.Cu") (net 6))
   (via (at 162.3 101.3) (size 0.8) (drill 0.4) (layers "F.Cu" "B.Cu") (net 6))
   (via (at 144.2 91.5) (size 0.8) (drill 0.4) (layers "F.Cu" "B.Cu") (net 6))
@@
   (segment (start 127 69.525) (end 131.88 74.405) (width 0.25) (layer "F.Cu") (net 30))
   (segment (start 127 67.31) (end 127 69.525) (width 0.25) (layer "F.Cu") (net 30))
-  (segment (start 135.128 101.092) (end 136.308 101.092) (width 0.25) (layer "F.Cu") (net 31))
-  (segment (start 137.795 99.605) (end 137.795 98.235) (width 0.25) (layer "F.Cu") (net 31))
+  (segment (start 136.652 71.12) (end 132.842 67.31) (width 0.25) (layer "F.Cu") (net 31))
+  (segment (start 136.508 101.092) (end 137.795 99.805) (width 0.25) (layer "F.Cu") (net 31))
+  (segment (start 132.842 67.31) (end 129.5 67.31) (width 0.25) (layer "F.Cu") (net 31))
+  (segment (start 129.54 82.804) (end 136.652 75.692) (width 0.25) (layer "F.Cu") (net 31))
+  (segment (start 135.128 101.092) (end 136.508 101.092) (width 0.25) (layer "F.Cu") (net 31))
   (segment (start 129.54 94.996) (end 129.54 82.804) (width 0.25) (layer "F.Cu") (net 31))
-  (segment (start 136.652 71.12) (end 132.842 67.31) (width 0.25) (layer "F.Cu") (net 31))
-  (segment (start 129.54 82.804) (end 136.652 75.692) (width 0.25) (layer "F.Cu") (net 31))
-  (segment (start 132.842 67.31) (end 129.5 67.31) (width 0.25) (layer "F.Cu") (net 31))
-  (segment (start 136.308 101.092) (end 137.795 99.605) (width 0.25) (layer "F.Cu") (net 31))
+  (segment (start 137.795 99.805) (end 137.795 98.235) (width 0.25) (layer "F.Cu") (net 31))
   (segment (start 136.652 75.692) (end 136.652 71.12) (width 0.25) (layer "F.Cu") (net 31))
   (via (at 135.128 101.092) (size 0.8) (drill 0.4) (layers "F.Cu" "B.Cu") (net 31))
   (via (at 129.54 94.996) (size 0.8) (drill 0.4) (layers "F.Cu" "B.Cu") (net 31))
-  (segment (start 134.62 101.092) (end 129.54 96.012) (width 0.25) (layer "B.Cu") (net 31))
   (segment (start 135.128 101.092) (end 134.62 101.092) (width 0.25) (layer "B.Cu") (net 31))
   (segment (start 129.54 96.012) (end 129.54 94.996) (width 0.25) (layer "B.Cu") (net 31))
+  (segment (start 112.285 102.93) (end 116.6 98.615) (width 0.25) (layer "B.Cu") (net 31))
+  (segment (start 134.62 101.092) (end 129.54 96.012) (width 0.25) (layer "B.Cu") (net 31))
+  (segment (start 114.94 81.34) (end 112.285 81.34) (width 0.25) (layer "B.Cu") (net 31))
+  (segment (start 116.6 98.615) (end 116.6 83) (width 0.25) (layer "B.Cu") (net 31))
+  (segment (start 116.6 83) (end 114.94 81.34) (width 0.25) (layer "B.Cu") (net 31))
   (segment (start 109.22 107.95) (end 109.24 107.93) (width 0.25) (layer "F.Cu") (net 32))
   (segment (start 112.285 86.34) (end 110.51 86.34) (width 0.25) (layer "F.Cu") (net 32))
